Commit message: add: config cartesian_controllers/cartesian_compliant_controller

File: franka_description/robots/panda_arm.xacro (robot description, xacro)
@@ -310,4 +310,11 @@
       <child link="${arm_id}_link8"/>
     </joint>
+    <!-- F/T SENSOR -->
+    <link name="${arm_id}_ft_sensor" />
+    <joint name="${arm_id}_ft_sensor_joint" type="fixed">
+      <origin rpy="0 0 3.14" xyz="0 0 0.102" />
+      <parent link="${arm_id}_link8" />
+      <child link="${arm_id}_ft_sensor" />
+    </joint>
   </xacro:macro>
 </robot>

Commit message: return to default panda_arm.xacro

File: franka_description/robots/panda_arm.xacro (robot description, xacro)
@@ -310,11 +310,4 @@
       <child link="${arm_id}_link8"/>
     </joint>
-    <!-- F/T SENSOR -->
-    <link name="${arm_id}_ft_sensor" />
-    <joint name="${arm_id}_ft_sensor_joint" type="fixed">
-      <origin rpy="0 0 3.14" xyz="0 0 0.102" />
-      <parent link="${arm_id}_link8" />
-      <child link="${arm_id}_ft_sensor" />
-    </joint>
   </xacro:macro>
 </robot>
